File: pcb/soic2dip16/soic2dip16.kicad_pcb (KiCad board)
At the start: 2 copper layers, 0 parts

Commit message: SOIC to DIP 16 Adapter PCB example
Parts:
- added J1: DIP, Package_DIP:DIP-16_W7.62mm_LongPads, F.Cu at (54.7, 29.4)
- added J2: SOIC, Package_SO:SOIC-16_3.9x9.9mm_P1.27mm, F.Cu at (70.9, 38.4)
Routing:
- net Net-(J1-Pin_12): track 0.00 -> 18.5 mm
- net Net-(J1-Pin_13): track 0.00 -> 17.8 mm
- net Net-(J1-Pin_8): track 0.00 -> 17.0 mm, vias 0 -> 1
- net Net-(J1-Pin_2): track 0.00 -> 17.0 mm, vias 0 -> 1
- net Net-(J1-Pin_14): track 0.00 -> 16.6 mm
- net Net-(J1-Pin_11): track 0.00 -> 16.4 mm
- net Net-(J1-Pin_7): track 0.00 -> 16.2 mm, vias 0 -> 1
- net Net-(J1-Pin_10): track 0.00 -> 15.7 mm
- net Net-(J1-Pin_1): track 0.00 -> 15.6 mm, vias 0 -> 1
- net Net-(J1-Pin_15): track 0.00 -> 15.5 mm
- net Net-(J1-Pin_6): track 0.00 -> 15.3 mm, vias 0 -> 1
- net Net-(J1-Pin_5): track 0.00 -> 14.9 mm, vias 0 -> 1
- net Net-(J1-Pin_4): track 0.00 -> 14.8 mm, vias 0 -> 1
- net Net-(J1-Pin_3): track 0.00 -> 14.5 mm, vias 0 -> 1
- net Net-(J1-Pin_9): track 0.00 -> 14.5 mm
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Other:
- board outline added: 23.5 x 23.5 mm
