File: circuits/mat464v1/concepts/mat464psv1/mat464psv1.kicad_pcb (KiCad board)
At the start: 2 copper layers, 23 parts, among them J1 5V, J2 GND, J3 +VDC, J4 GND VDC, J5 -VDC, J6 Zero crossing det, Q1 BC547, Q2 BC547, Q3 BC547, U1 L7805

Commit message: Update the modern AT464 concepts
Parts:
- added J10: NEUTRAL, Connector_Pin:Pin_D1.1mm_L8.5mm_W2.5mm_FlatFork, F.Cu at (178.3, 91.7)
- added J7: VDC A, Connector_Pin:Pin_D1.1mm_L8.5mm_W2.5mm_FlatFork, F.Cu at (178.6, 71.2)
- added J8: VDC B, Connector_Pin:Pin_D1.1mm_L8.5mm_W2.5mm_FlatFork, F.Cu at (178.3, 81.4)
- added J9: LIVE, Connector_Pin:Pin_D1.1mm_L8.5mm_W2.5mm_FlatFork, F.Cu at (178.8, 61.0)
- moved J5 59.6 mm to (154.4, 59.2)
- moved J4 48.6 mm to (144.0, 59.2)
- moved C5 40.5 mm to (117.9, 67.5), turned to 90 degrees
- moved R1 39.5 mm to (135.9, 93.0), turned to -90 degrees
- moved U1 38.3 mm to (126.0, 69.6), turned to -90 degrees
- moved Q3 37.8 mm to (145.0, 82.5), turned to 180 degrees
- moved J3 37.6 mm to (133.6, 59.2)
- moved Q2 34.3 mm to (137.2, 82.5), turned to 180 degrees
- moved R6 34.2 mm to (117.8, 74.7)
- moved Q1 33.3 mm to (129.3, 82.5), turned to 180 degrees
- moved R2 31.8 mm to (142.5, 103.1), turned to 90 degrees
- moved C4 30.7 mm to (110.0, 67.6), turned to 90 degrees
- moved R5 26.0 mm to (110.0, 74.7)
- moved J2 10.7 mm to (103.1, 66.8)
- moved J6 5.85 mm to (170.7, 103.1)
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Routing:
- net GND: track 0.00 -> 159.0 mm, vias 0 -> 4
- net +VDC: track 0.00 -> 72.4 mm, vias 0 -> 2
- net Net-(J9-Pin_1): track 0.00 -> 69.0 mm
- net Net-(Q1-E): track 0.00 -> 44.5 mm, vias 0 -> 2
- net Net-(J6-Pin_1): track 0.00 -> 39.4 mm
- net Net-(Q1-C): track 0.00 -> 30.2 mm
- net Net-(D1-K): track 0.00 -> 20.9 mm
- net -VDC: track 0.00 -> 17.2 mm
- net Net-(U1-OUT): track 0.00 -> 12.6 mm
- net Net-(C4-Pad1): track 0.00 -> 10.7 mm
- net Net-(J1-Pin_1): track 0.00 -> 5.28 mm
Other:
- board outline added: 83.6 x 51.8 mm
